Commit message: Clean up dead files, refactor training with DummyVecEnv, update demo video
Co-Authored-By: Claude Opus 4.7 <noreply@anthropic.com>

File: assets/franka_panda/robots/panda_arm.urdf (robot description, URDF)
Before this commit: robot panda, 9 links, 8 joints
Links:
- added link peg_tip_frame
Joints:
- added joint peg_tip_joint: type fixed, parent panda_link8, child peg_tip_frame, origin xyz=0 0 0.185 rpy=0 0 0
